Commit message: Aggiunto il package fanuc_moveit_config

File: esercizio3_ws/src/fanuc_description/robot/fanuc.xacro (robot description, xacro)
@@ -78,5 +78,5 @@
         <!--Link properties-->
         <visual>
-            <origin xyz="-1.315 0 0.15" rpy="-${pi/2} 0 -${pi/2}" />
+            <origin xyz="-1.315 0.15 0" rpy="-${pi/2} 0 -${pi/2}" />
             <geometry>
                 <mesh filename="package://fanuc_description/meshes/visual/link_3.dae" />
@@ -85,5 +85,5 @@
         </visual>
         <collision>
-            <origin xyz="-1.315 0 0.15" rpy="-${pi/2} 0 ${pi/2}" />
+            <origin xyz="-1.315 0.15 0" rpy="-${pi/2} 0 ${pi/2}" />
             <geometry>
                 <mesh filename="package://fanuc_description/meshes/collision/link_3.stl" />
